File: shield_controller/Controller.sch (KiCad schematic (older format))
At the start: 16 parts, among them J1 Input Power, J2 Track, J3 DCC, J4 Calc, U1 LM7805_TO220, U2 LMD18200T

Commit message: Updating Christopher's shield controller to current fabbed version
Parts:
- added J5: EBrake, Pin_Headers:Pin_Header_Straight_1x02_Pitch2.54mm, symbol conn:CONN_01X02
- added PP1: CR, Wire_Pads:SolderWirePad_single_0-8mmDrill, symbol conn:CONN_01X01
- added PP2: CW, Wire_Pads:SolderWirePad_single_0-8mmDrill, symbol conn:CONN_01X01
- added PP3: DIR, Wire_Pads:SolderWirePad_single_0-8mmDrill, symbol conn:CONN_01X01
- added PP4: CS, Wire_Pads:SolderWirePad_single_0-8mmDrill, symbol conn:CONN_01X01
- added PP5: +5V, Wire_Pads:SolderWirePad_single_0-8mmDrill, symbol conn:CONN_01X01
- added PP6: GND, Wire_Pads:SolderWirePad_single_0-8mmDrill, symbol conn:CONN_01X01
- C1, C2, C3: symbol C -> device:C
- C4: symbol CP1_Small -> device:CP1_Small
- C5: symbol C_Small -> device:C_Small
- D1: symbol LED-RESCUE-Controller -> Controller-rescue:LED-RESCUE-Controller
- J1: symbol CONN_01X04 -> conn:CONN_01X04
- J2, J3: symbol CONN_01X02 -> conn:CONN_01X02
- J4: symbol CONN_01X03 -> conn:CONN_01X03
- R1, R2, R3: symbol R -> device:R
- SHIELD1: symbol ARDUINO_SHIELD -> freetronics_schematic:ARDUINO_SHIELD
- U1: symbol LM7805_TO220 -> regul:LM7805_TO220
- U2: symbol LMD18200T -> LMD18200T:LMD18200T
Connections:
- wire segments 50 -> 65
- no-connect marks 0 -> 1
Other:
- note added: "Prototyping Breakout Area"
